File: hardware/raspberrycanshield.kicad_pcb (KiCad board)
At the start: 2 copper layers, 88 x 56 mm, 68 parts, among them J101 I2C, J102 USART, J103 Conn_01x06, J401 Raspberry_Pi_2_3, J501 RJ45, J502 RJ45, U201 MCP2515-xSO, U202 MCP2551-I/SN, U301 LM7805, Y201 16MHz

Commit message: Silkscreen updated with JLC. Finished.
Parts:
- removed H101, H102, H103, H104: ~, MountingHole:MountingHole_3.2mm_M3
- removed SYM102: SYM_Magnet_Large, rasp3:raspberrypi_2_3
- added R103: 10k, Resistor_SMD:R_0603_1608Metric_Pad0.98x0.95mm_HandSolder, F.Cu at (128.9, 107.8)
- added R104: 10k, Resistor_SMD:R_0603_1608Metric_Pad0.98x0.95mm_HandSolder, F.Cu at (120.0, 107.8)
- LOGO101: moved to B.Cu
- moved LOGO101 158.1 mm to (147.9, 66.6), turned to 90 degrees
- moved C302 55.7 mm to (131.6, 79.1)
- moved C401 55.7 mm to (175.1, 109.8)
- moved J401 55.7 mm to (172.3, 112.7)
- moved TP206 55.7 mm to (143.0, 96.6)
- moved R101 55.7 mm to (101.8, 75.8)
- moved TP101 55.7 mm to (96.9, 93.2)
- moved TP207 55.7 mm to (146.5, 96.6)
- moved C101 55.7 mm to (100.7, 105.2)
- moved C201 55.7 mm to (140.0, 98.3)
- moved C202 55.7 mm to (140.0, 101.9)
- moved C203 55.7 mm to (151.8, 89.3)
- moved C205 55.7 mm to (133.3, 88.1)
- moved C301 55.7 mm to (129.2, 80.1)
- moved C304 55.7 mm to (147.1, 74.0)
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Routing:
- net +3V3: track 128.7 -> 136.2 mm
- net /MCU/SDA: track 145.0 -> 148.5 mm
- net /MCU/SCL: track 139.7 -> 141.9 mm
- net GND: vias 5 -> 7
Other:
- board text added: "Designed by Zenite Solar Boat Team"
- board text added: "JLCJLCJLCJLC"
- board text added: "github.com/ZeniteSolar/MSC22"
